File: schematics/sensors.kicad_sch (KiCad schematic)
At the start: 15 parts, among them U10 ArducamOV2640, U11 WMM7027ATSN1, U7 VL53L7CX, U9 MPU-6500

Commit message: Fixed mistake in battery bypass circuit.
Other:
- note added: "SDI = MOSI SDO = MISO"
Changed lines of the file:
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@@
+		)
+	)
+	(text "SDI = MOSI\nSDO = MISO"
+		(exclude_from_sim no)
+		(at 169.418 83.312 0)
+		(effects
+			(font
+				(size 1.27 1.27)
+			)
 		)
 	)
@@
 	)
 	(global_label "SPI_SDI"
-		(shape output)
+		(shape input)
 		(at 148.59 58.42 180)
 		(fields_autoplaced yes)
@@
 	)
 	(global_label "SPI_SDO"
-		(shape input)
+		(shape output)
 		(at 189.23 55.88 0)
 		(fields_autoplaced yes)
